File: PCB/PCB/Step_Down_Module.sch (EAGLE design)
At the start: 42 parts, among them Q1 TPH2900ENH

Commit message: PCB changes, added through hole part for RP, fixed pot error
Parts:
- RP: device rcl:R-EU_R0805 -> SparkFun-Resistors:RESISTORAXIAL-0.3
Connections:
- net GND: no longer V_ADJ.E
- net N$6: now also RP.1; no longer RP.2
- net VOUT: now also RP.2; no longer RP.1
Changed lines of the file:
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@@
 <layer number="230" name="230bmp" color="7" fill="1" visible="yes" active="yes"/>
 <layer number="231" name="231bmp" color="7" fill="1" visible="yes" active="yes"/>
+<layer number="232" name="Eagle3D_PG2" color="7" fill="1" visible="yes" active="yes"/>
+<layer number="233" name="Eagle3D_PG3" color="7" fill="1" visible="yes" active="yes"/>
 <layer number="248" name="Housing" color="7" fill="1" visible="yes" active="yes"/>
 <layer number="249" name="Edge" color="7" fill="1" visible="yes" active="yes"/>
@@
 <part name="CS" library="rcl" library_urn="urn:adsk.eagle:library:334" deviceset="C-EU" device="C0805" package3d_urn="urn:adsk.eagle:package:23617/2" value="0.01uF"/>
 <part name="RS" library="rcl" library_urn="urn:adsk.eagle:library:334" deviceset="R-EU_" device="R0805" package3d_urn="urn:adsk.eagle:package:23553/2" value="270k"/>
-<part name="RP" library="rcl" library_urn="urn:adsk.eagle:library:334" deviceset="R-EU_" device="R0805" package3d_urn="urn:adsk.eagle:package:23553/2" value="10000k"/>
 <part name="RFBT" library="rcl" library_urn="urn:adsk.eagle:library:334" deviceset="R-EU_" device="R0805" package3d_urn="urn:adsk.eagle:package:23553/2" value="180k"/>
 <part name="RFBB" library="rcl" library_urn="urn:adsk.eagle:library:334" deviceset="R-EU_" device="R0805" package3d_urn="urn:adsk.eagle:package:23553/2" value="4.7k"/>
@@
 <part name="COC1" library="rcl" library_urn="urn:adsk.eagle:library:334" deviceset="CPOL-EU" device="E5-5" package3d_urn="urn:adsk.eagle:package:23367/1" value="22uF"/>
 <part name="COB1" library="rcl" library_urn="urn:adsk.eagle:library:334" deviceset="CPOL-EU" device="E5-10.5" package3d_urn="urn:adsk.eagle:package:23372/1" value="150uF"/>
-<part name="GND20" library="SparkFun-PowerSymbols" library_urn="urn:adsk.eagle:library:530" deviceset="GND" device=""/>
 <part name="RS2" library="rcl" library_urn="urn:adsk.eagle:library:334" deviceset="R-EU_" device="R0805" package3d_urn="urn:adsk.eagle:package:23553/2" value="10k"/>
 <part name="CINC1" library="rcl" library_urn="urn:adsk.eagle:library:334" deviceset="C-EU" device="150-084X183" package3d_urn="urn:adsk.eagle:package:23658/1" value=".47uF"/>
@@
 <part name="GND24" library="SparkFun-PowerSymbols" library_urn="urn:adsk.eagle:library:530" deviceset="GND" device=""/>
 <part name="V_ADJ" library="pot" deviceset="RM065" device="" value="10k"/>
+<part name="RP" library="SparkFun-Resistors" deviceset="RESISTOR" device="AXIAL-0.3" value="10000k"/>
 </parts>
 <sheets>
@@
 <attribute name="VALUE" x="74.422" y="64.77" size="1.778" layer="96" rot="R90"/>
 </instance>
-<instance part="RP" gate="G$1" x="81.28" y="50.8" smashed="yes" rot="R180">
-<attribute name="NAME" x="85.09" y="49.3014" size="1.778" layer="95" rot="R180"/>
-<attribute name="VALUE" x="85.09" y="54.102" size="1.778" layer="96" rot="R180"/>
-</instance>
 <instance part="RFBT" gate="G$1" x="101.6" y="40.64" smashed="yes" rot="R90">
 <attribute name="NAME" x="100.1014" y="36.83" size="1.778" layer="95" rot="R90"/>
@@
 <attribute name="VALUE" x="138.303" y="66.5226" size="1.778" layer="96"/>
 </instance>
-<instance part="GND20" gate="1" x="106.68" y="50.8" smashed="yes">
-<attribute name="VALUE" x="106.68" y="50.546" size="1.778" layer="96" align="top-center"/>
-</instance>
 <instance part="RS2" gate="G$1" x="71.12" y="55.88" smashed="yes" rot="R90">
 <attribute name="NAME" x="69.6214" y="52.07" size="1.778" layer="95" rot="R90"/>
@@
 <attribute name="NAME" x="112.649" y="64.77" size="1.778" layer="95" rot="R270"/>
 <attribute name="VALUE" x="110.49" y="64.77" size="1.778" layer="96" rot="R270"/>
+</instance>
+<instance part="RP" gate="G$1" x="78.74" y="50.8" smashed="yes">
+<attribute name="NAME" x="78.74" y="52.324" size="1.778" layer="95" font="vector" align="bottom-center"/>
+<attribute name="VALUE" x="78.74" y="49.276" size="1.778" layer="96" font="vector" align="top-center"/>
 </instance>
 </instances>
@@
 <wire x1="106.68" y1="66.04" x2="106.68" y2="73.66" width="0.1524" layer="91"/>
 <pinref part="U$1" gate="G$1" pin="SENSE-"/>
-<pinref part="RP" gate="G$1" pin="1"/>
-<wire x1="86.36" y1="50.8" x2="86.36" y2="43.18" width="0.1524" layer="91"/>
 <wire x1="86.36" y1="43.18" x2="50.8" y2="43.18" width="0.1524" layer="91"/>
 <pinref part="CS" gate="G$1" pin="1"/>
 <junction x="50.8" y="43.18"/>
 <wire x1="50.8" y1="43.18" x2="38.1" y2="43.18" width="0.1524" layer="91"/>
+<wire x1="86.36" y1="43.18" x2="86.36" y2="50.8" width="0.1524" layer="91"/>
 <wire x1="86.36" y1="50.8" x2="86.36" y2="73.66" width="0.1524" layer="91"/>
-<junction x="86.36" y="50.8"/>
 <wire x1="106.68" y1="73.66" x2="91.44" y2="73.66" width="0.1524" layer="91"/>
 <pinref part="L1" gate="G$1" pin="P$2"/>
@@
 <wire x1="91.44" y1="43.18" x2="91.44" y2="73.66" width="0.1524" layer="91"/>
 <junction x="91.44" y="73.66"/>
+<pinref part="RP" gate="G$1" pin="2"/>
+<wire x1="83.82" y1="50.8" x2="86.36" y2="50.8" width="0.1524" layer="91"/>
+<junction x="86.36" y="50.8"/>
 </segment>
 <segment>
@@
 <junction x="50.8" y="50.8"/>
 <pinref part="RS2" gate="G$1" pin="1"/>
-<pinref part="RP" gate="G$1" pin="2"/>
-<wire x1="76.2" y1="50.8" x2="71.12" y2="50.8" width="0.1524" layer="91"/>
+<wire x1="73.66" y1="50.8" x2="71.12" y2="50.8" width="0.1524" layer="91"/>
 <junction x="71.12" y="50.8"/>
+<pinref part="RP" gate="G$1" pin="1"/>
 </segment>
 </net>
@@
 </segment>
 <segment>
-<pinref part="GND20" gate="1" pin="GND"/>
-<wire x1="106.68" y1="55.88" x2="106.68" y2="53.34" width="0.1524" layer="91"/>
-<pinref part="V_ADJ" gate="G$1" pin="E"/>
-</segment>
-<segment>
